File: LCD Project/LCD_Project/Switch Board/LCD_Project.kicad_sch (KiCad schematic)
At the start: 24 parts, among them IC1 REG1117-5, J1 353630460, U1 Teensy4.0, U2 VOM618A-3T, U4 VOM618A-3T, U5 VOM618A-3T, U6 VOM618A-3T

Commit message: Add files via upload
Parts:
- removed J1: 353630460, 353630460:CON_353630460, symbol 353630460:353630460
- removed R7: R_250, Resistor_SMD:R_0805_2012Metric, symbol Device:R_US
- removed R8: R_110, Resistor_SMD:R_0805_2012Metric, symbol Device:R_US
- added C3, C4: C0805C104Z3VACTU, C0805C104Z3VACTU:CAPC2012X88N, symbol C0805C104Z3VACTU:C0805C104Z3VACTU
- added J1: DT15-4P, DT15-4P:TE_DT15-4P, symbol DT15-4P:DT15-4P
- added U3: MIC5365-1.3YC5-TR, MIC5365-1.3YC5-TR:SOT65P210X110-5N, symbol MIC5365-1.3YC5-TR:MIC5365-1.3YC5-TR
Connections:
- net +12V: now also C4.1, J1.1, U3.1 (VIN), U3.3 (EN)
- net GND: now also C3.2, C4.2, J1.4, U3.2 (GND)
- net at U1.21 (14_A0_TX3_SPDIF_OUT): now also J1.2
- net at U1.22 (15_A1_RX3_SPDIF_IN): now also J1.3
- net +3.7V: no longer names the net of DS1.3_1 (V0), DS1.3_2 (V0)
- new net +1.3V: C3.1, U3.5 (VOUT)
- no-connect marks 37 -> 38
